Commit message: works

File: urdf/sdnova.urdf (robot description, URDF)
Before this commit: robot sdnova, 2 links, 1 joints
Links:
- removed link link_imu
- added link body_link, mass ${base_mass}; collision box size=${base_length} ${base_width} ${base_height}; visual box size=${base_length} ${base_width} ${base_height}
- added link imu_link
- added link lidar_link, mass 0.125; collision cylinder length=0.055 radius=0.0508; visual cylinder length=0.055 radius=0.0508
- link base_link: mass ${base_mass} -> None; geometry 
Joints:
- added joint base_joint: type fixed, parent base_link, child body_link, origin xyz=0 0 0 rpy=0 0 0
- added joint lidar_joint: type fixed, parent body_link, child lidar_link, origin xyz=0 0 ${base_height/2} rpy=0 0 0
- joint joint_imu: child link_imu -> imu_link; parent base_link -> body_link

Commit message: update world

File: urdf/sdnova.urdf (robot description, URDF)
Before this commit: robot sdnova, 4 links, 3 joints
Links:
- link lidar_link: geometry collision cylinder length=0.05 radius=0.0508; visual cylinder length=0.05 radius=0.0508

Commit message: new world &fix lidar bug

File: urdf/sdnova.urdf (robot description, URDF)
Before this commit: robot sdnova, 4 links, 3 joints
Joints:
- joint lidar_joint: origin xyz=0 0 ${base_height/2} rpy=0 0 0 -> xyz=0 0 ${base_height/2 + 0.025} rpy=0 0 0

Commit message: fix urdf

File: urdf/sdnova.urdf (robot description, URDF)
Before this commit: robot sdnova, 4 links, 3 joints
Links:
- removed link body_link
- added link base_footprint
- link base_link: mass None -> ${base_mass}; geometry collision box size=${base_length} ${base_width} ${base_height}; visual box size=${base_length} ${base_width} ${base_height}
Joints:
- joint base_joint: child body_link -> base_link; origin xyz=0 0 0 rpy=0 0 0 -> xyz=0 0 ${base_height/2} rpy=0 0 0; parent base_link -> base_footprint
- joint joint_imu: parent body_link -> base_link
- joint lidar_joint: parent body_link -> base_link

Commit message: 从urdf 赋值 option

File: urdf/sdnova.urdf (robot description, URDF)
Before this commit: robot sdnova, 4 links, 3 joints
Links:
- link base_link: mass ${base_mass} -> ${body_mass}; geometry collision box size=${body_length} ${body_width} ${body_height}; visual box size=${body_length} ${body_width} ${body_height}
Joints:
- joint base_joint: origin xyz=0 0 ${base_height/2} rpy=0 0 0 -> xyz=0 0 ${body_height/2} rpy=0 0 0
- joint lidar_joint: origin xyz=0 0 ${base_height/2 + 0.025} rpy=0 0 0 -> xyz=0 0 ${body_height/2 + 0.025} rpy=0 0 0
